Commit message: LiDAR yaw from bench test

File: hospital_robot_description/urdf/robot.urdf.xacro (robot description, xacro)
@@ -53,5 +53,5 @@
   <xacro:property name="lidar_y"      value="0.209025"/>
   <xacro:property name="lidar_z"      value="0.3209"/>
-  <xacro:property name="lidar_yaw"    value="0.0"/>
+  <xacro:property name="lidar_yaw"    value="-1.5708"/>
   <xacro:property name="lidar_radius" value="0.038"/>
   <xacro:property name="lidar_height" value="0.04"/>

Commit message: Phase 9: lidar_gaze + eyes (hospital_robot_hri)

File: hospital_robot_description/urdf/robot.urdf.xacro (robot description, xacro)
@@ -21,9 +21,9 @@
   <!-- VERIFY: vertical distance from the ground up to your Z=0 origin
        plane. See README_NEXT_STEPS.md Part A. -->
-  <xacro:property name="origin_ground_clearance" value="0.02"/>
+  <xacro:property name="origin_ground_clearance" value="0.051"/>
   <!-- Drive wheels -->
   <xacro:property name="wheel_radius"     value="0.072"/>
   <xacro:property name="wheel_width"      value="0.029"/>
-  <xacro:property name="wheel_separation" value="0.260"/>
+  <xacro:property name="wheel_separation" value="0.245"/>
   <xacro:property name="wheel_x"          value="0.176982"/>
   <xacro:property name="wheel_mass"       value="0.34"/>
@@ -35,6 +35,6 @@
        base_width/wheel_separation math here, that's what was
        causing the misalignment. -->
-  <xacro:property name="wheel_left_y"     value="0.35"/>
-  <xacro:property name="wheel_right_y"    value="0.09"/>
+  <xacro:property name="wheel_left_y"     value="0.3315"/>
+  <xacro:property name="wheel_right_y"    value="0.0865"/>
   <!-- Casters — you have FOUR (one per corner), not one. Positions are
        your raw Measurements.md values, used directly. -->
@@ -50,7 +50,7 @@
   <xacro:property name="caster4_y" value="0.381794"/>
   <!-- LiDAR -->
-  <xacro:property name="lidar_x"      value="0.222025"/>
-  <xacro:property name="lidar_y"      value="0.209025"/>
-  <xacro:property name="lidar_z"      value="0.3209"/>
+  <xacro:property name="lidar_x"      value="0.238"/>
+  <xacro:property name="lidar_y"      value="0.210"/>
+  <xacro:property name="lidar_z"      value="0.299"/>
   <xacro:property name="lidar_yaw"    value="-1.5708"/>
   <xacro:property name="lidar_radius" value="0.038"/>
@@ -63,5 +63,5 @@
   <xacro:property name="column_side"   value="0.08"/>
   <xacro:property name="column_length" value="0.677971"/>  <!-- VERIFY: derived, see README Part B -->
-  <xacro:property name="column_travel" value="0.380"/>
+  <xacro:property name="column_travel" value="0.300"/>
   <xacro:property name="column_mass"   value="1.5"/>
   <!-- Camera — expressed relative to column_link's own origin (derived
@@ -73,7 +73,7 @@
   <xacro:property name="camera_mass"  value="0.05"/>
   <!-- IMU -->
-  <xacro:property name="imu_x" value="0.0895"/>
-  <xacro:property name="imu_y" value="0.207"/>
-  <xacro:property name="imu_z" value="0.275501"/>
+  <xacro:property name="imu_x" value="-0.052"/>
+  <xacro:property name="imu_y" value="-0.066"/>
+  <xacro:property name="imu_z" value="0.497"/>
   <!-- Mesh correction: your Inventor parts are Y-up, ROS/RViz is Z-up.
        rpy = "${pi/2} 0 0" fixes that (Inventor Y -> RViz Z, up).
@@ -133,5 +133,5 @@
     <parent link="base_footprint"/>
     <child  link="base_link"/>
-    <origin xyz="-0.176982 -0.22 ${origin_ground_clearance}" rpy="0 0 0"/>
+    <origin xyz="${-wheel_x} ${-(wheel_left_y + wheel_right_y)/2} ${origin_ground_clearance}" rpy="0 0 0"/>
   </joint>
   <!-- ================= CHASSIS ================= -->
@@ -295,5 +295,5 @@
   <!-- ================= IMU ================= -->
   <joint name="imu_joint" type="fixed">
-    <parent link="base_link"/>
+    <parent link="column_link"/>
     <child  link="imu_link"/>
     <origin xyz="${imu_x} ${imu_y} ${imu_z}" rpy="0 0 0"/>
